File: train1/ESP32.kicad_sch (KiCad schematic)
At the start: 14 parts, among them J5 header-2.54mm-7p, SW1 tactileSW/4.2x3.3, SW2 tactileSW/4.2x3.3, U10 ESP32-WROOM-32E

Commit message: fix(repo): delete backup file
Parts:
- C26, C29: Part number  (none) -> LM7805CT; manafacture (none) -> onsemi
Connections:
- net ESP.SCL: now also U10.33 (IO21); no longer U10.36 (IO22)
- net ESP.SDA: now also U10.36 (IO22); no longer U10.33 (IO21)
- net ESP.DN: now reaches U10.13 (IO14)
- net ESP.DP: now reaches U10.16 (IO13)
- no-connect marks 12 -> 10
Other:
- moved on the sheet: C26, C27, C28, C29, C31, J5, R30, R31, R32, R33, SW1, SW2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
