File: train1/train1.kicad_sch (KiCad schematic)
At the start: 0 parts

Commit message: fix(repo): delete backup file
Other:
- note added: "SETUP PHẦN MỀM CÀI PLUGIN JLC và IBOM =================THIẾT KẾ SẢN PHẨM==================== NGHIÊN CỨU SẢN PHẨM MẪU CHỌN LINH KIỆN =================GIAI ĐOẠN PROTOTILE================== SYMBOL + FOOTPRINT ------------ tạo symbol - tạo symbol - cấu hình chân - symbol nhiều part - link symbol nhanh SCHEMATIC ------------------- hướng dẫn thêm thư viện, global và project hướng dẫn lấy linh kiện hướ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"
- note removed: "SETUP PHẦN MỀM CÀI PLUGIN JLC và IBOM =================THIẾT KẾ SẢN PHẨM==================== NGHIÊN CỨU SẢN PHẨM MẪU CHỌN LINH KIỆN =================GIAI ĐOẠN PROTOTILE================== SCHEMATIC ------------------- hướng dẫn thêm thư viện, global và project hướng dẫn lấy linh kiện hướng dẫn định nghĩa bus i2c, spi, bus số (demo vẽ insert) hướng dẫn dùng netclass(định nghĩa class, màu mè cho cla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"
